File: IMX219_4lane/imx219_4lane/imx219_4lane.kicad_sch (KiCad schematic)
At the start: 25 parts, among them J1 DF37NC-30DS-0.4V, J2 FPC 28 pin connector, Q3 NTZD3154N, U1 AMPM, U2 LM3670MF, U3 AP7331, U4 AP7331

Commit message: flip connector -.-
Parts:
- added TP1, TP2, TP3, TP4, TP5, TP6: TestPoint, unsurv_offline_pcb_footprints:TestPoint_Pad_D0.7mm, symbol Connector:TestPoint
Connections:
- net +1V2: now also TP2.1
- net +1V8: now also TP1.1
- net +5V: now also J2.2 (Pin_2), J2.3 (Pin_3), J2.4 (Pin_4); no longer J2.25 (Pin_25), J2.26 (Pin_26), J2.27 (Pin_27)
- net GND: now also J2.25 (Pin_25), TP5.1; no longer J2.4 (Pin_4)
- net I2C_SCL_3V3: now also J2.9 (Pin_9); no longer J2.20 (Pin_20)
- net I2C_SDA_3V3: now also J2.8 (Pin_8); no longer J2.21 (Pin_21)
- net MCLK: now also TP6.1
- net MIPI_CLK_N: now also J2.20 (Pin_20); no longer J2.9 (Pin_9)
- net MIPI_CLK_P: now also J2.21 (Pin_21); no longer J2.8 (Pin_8)
- net MIPI_DATA_0_N: now also J2.14 (Pin_14); no longer J2.15 (Pin_15)
- net MIPI_DATA_0_P: now also J2.15 (Pin_15); no longer J2.14 (Pin_14)
- net MIPI_DATA_1_N: now also J2.17 (Pin_17); no longer J2.12 (Pin_12)
- net MIPI_DATA_1_P: now also J2.18 (Pin_18); no longer J2.11 (Pin_11)
- net MIPI_DATA_2_N: now also J2.23 (Pin_23); no longer J2.6 (Pin_6)
- net MIPI_DATA_2_P: now also J2.24 (Pin_24); no longer J2.5 (Pin_5)
- net MIPI_DATA_3_N: now also J2.26 (Pin_26); no longer J2.3 (Pin_3)
- net MIPI_DATA_3_P: now also J2.27 (Pin_27); no longer J2.2 (Pin_2)
- net SAI2_RXD0: now also J2.6 (Pin_6); no longer J2.23 (Pin_23)
- net SAI2_TXC: now also J2.11 (Pin_11); no longer J2.18 (Pin_18)
- net SAI2_TXD0: now also J2.5 (Pin_5); no longer J2.24 (Pin_24)
- net SAI2_TXFS: now also J2.12 (Pin_12); no longer J2.17 (Pin_17)
- net SCL_1V8: now also TP4.1
- net SDA_1V8: now also TP3.1
Other:
- moved on the sheet: J2
